File: Hardware Files/PacketVis.kicad_pcb (KiCad board)
At the start: 2 copper layers, 59 x 44.5 mm, 36 parts, among them J1 USB_B_Micro, J2 Conn_01x04, SW1 SW_Push_Dual, SW2 SW_SPST, SW3 SW_SPST, U1 3.3V 1A, U2 74HC595, U3 ESP-WROOM-02D

Commit message: Change LEDs to source current from shift register, unroute most tracks
Parts:
- U2: footprint PacketVis_Footprints:SOIC-16 -> Package_SO:SOIC-16_3.9x9.9mm_P1.27mm
- moved D8 18.0 mm to (236.2, 83.5), turned to 0 degrees
- moved R9 18.0 mm to (231.2, 83.5)
- moved D1 17.0 mm to (236.2, 101.0), turned to 0 degrees
- moved R2 17.0 mm to (231.2, 101.0)
- moved D7 13.0 mm to (236.2, 86.0), turned to 0 degrees
- moved R8 13.0 mm to (231.2, 86.0)
- moved D2 12.0 mm to (236.2, 98.5), turned to 0 degrees
- moved R3 12.0 mm to (231.2, 98.5)
- moved D6 8.02 mm to (236.2, 88.5), turned to 0 degrees
- moved R7 8.01 mm to (231.2, 88.5)
- moved D3 7.02 mm to (236.2, 96.0), turned to 0 degrees
- moved R4 7.01 mm to (231.2, 96.0)
- moved U2 3.34 mm to (223.6, 87.6), turned to 180 degrees
- moved C3 3.18 mm to (194.9, 100.2), turned to 90 degrees
- moved D5 3.05 mm to (236.2, 91.0), turned to 0 degrees
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Connections:
- D1 pad 1: /LED_1 -> Net-(D1-Pad1)
- D1 pad 2: Net-(D1-Pad2) -> /LED_1
- D2 pad 1: /LED_2 -> Net-(D2-Pad1)
- D2 pad 2: Net-(D2-Pad2) -> /LED_2
- D3 pad 1: /LED_3 -> Net-(D3-Pad1)
- D3 pad 2: Net-(D3-Pad2) -> /LED_3
- D4 pad 1: /LED_4 -> Net-(D4-Pad1)
- D4 pad 2: Net-(D4-Pad2) -> /LED_4
- D5 pad 1: /LED_5 -> Net-(D5-Pad1)
- D5 pad 2: Net-(D5-Pad2) -> /LED_5
- D6 pad 1: /LED_6 -> Net-(D6-Pad1)
- D6 pad 2: Net-(D6-Pad2) -> /LED_6
- D7 pad 1: /LED_7 -> Net-(D7-Pad1)
- D7 pad 2: Net-(D7-Pad2) -> /LED_7
- D8 pad 1: /LED_8 -> Net-(D8-Pad1)
- D8 pad 2: Net-(D8-Pad2) -> /LED_8
- R2 pad 1: +3V3 -> GND
- R2 pad 2: Net-(D1-Pad2) -> Net-(D1-Pad1)
- R3 pad 1: +3V3 -> GND
- R3 pad 2: Net-(D2-Pad2) -> Net-(D2-Pad1)
- R4 pad 1: +3V3 -> GND
- R4 pad 2: Net-(D3-Pad2) -> Net-(D3-Pad1)
- R5 pad 1: +3V3 -> GND
- R5 pad 2: Net-(D4-Pad2) -> Net-(D4-Pad1)
- R6 pad 1: +3V3 -> GND
- R6 pad 2: Net-(D5-Pad2) -> Net-(D5-Pad1)
- R7 pad 1: +3V3 -> GND
- R7 pad 2: Net-(D6-Pad2) -> Net-(D6-Pad1)
- R8 pad 1: +3V3 -> GND
- R8 pad 2: Net-(D7-Pad2) -> Net-(D7-Pad1)
- R9 pad 1: +3V3 -> GND
- R9 pad 2: Net-(D8-Pad2) -> Net-(D8-Pad1)
Routing:
- net /SW_1: track 52.0 -> 0.00 mm, vias 2 -> 0
- net +3V3: track 40.9 -> 0.04 mm, vias 12 -> 6
- net /ESP_EN: track 35.6 -> 0.44 mm, vias 2 -> 0
- net +5V: track 28.4 -> 0.57 mm
- net /CLEAR: track 44.8 -> 22.6 mm
- net /OUTPUT_ENABLE: track 44.6 -> 25.6 mm
- net /LATCH: track 22.8 -> 5.17 mm, vias 2 -> 0
- net /CLOCK: track 37.1 -> 26.0 mm
- net /LED_1: track 14.2 -> 24.3 mm
- net /LED_8: track 25.7 -> 15.6 mm
- net /LED_7: track 25.2 -> 15.3 mm
- net /LED_6: track 24.7 -> 15.8 mm
- net /DATA: track 17.4 -> 8.69 mm
- net /LED_5: track 24.2 -> 16.3 mm
- net /LED_4: track 23.7 -> 16.8 mm
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- added copper zone on B.Cu, net GND
- removed copper zone on B.Cu, net +3V3
Other:
- board text added: "8Bit WiFi Visualizer"
- board text added: "A04"
- board text removed: "A03"
- board text removed: "ESP8266 8 Bit Vis"

Commit message: Update Routing
Parts:
- removed C1: 47pF, Capacitor_SMD:C_0805_2012Metric
- removed FB1: Ferrite_Bead, Inductor_SMD:L_0805_2012Metric
- moved R1 26.5 mm to (201.7, 101.5)
- moved R12 14.7 mm to (194.2, 92.5), turned to 270 degrees
- moved R10 9.85 mm to (199.2, 101.5)
- moved SW2 7.42 mm to (210.4, 104.8)
- moved SW3 7.42 mm to (210.4, 100.2)
- moved C4 2.02 mm to (194.2, 81.5)
- moved C5 2.02 mm to (196.7, 81.5)
- moved C3 1.46 mm to (194.2, 101.5)
- moved C2 1.35 mm to (196.7, 101.5)
- moved R11 1.00 mm to (194.2, 85.5)
- moved U1 0.56 mm to (196.7, 108.2)
- moved C6 0.50 mm to (196.7, 85.5)
- moved R13 0.50 mm to (196.7, 92.5)
Connections:
- J1 pad 1: Net-(C1-Pad1) -> +5V
Routing:
- net +3V3: track 0.04 -> 90.5 mm, vias 6 -> 8
- net /SW_1: track 0.00 -> 66.9 mm, vias 0 -> 2
- net /ESP_EN: track 0.44 -> 42.7 mm, vias 0 -> 2
- net +5V: track 0.57 -> 20.0 mm, vias 0 -> 1
- net /BOOT: track 17.6 -> 27.1 mm
- net Net-(R13-Pad1): track 0.00 -> 4.17 mm
- net /ESP_RX: track 34.9 -> 36.7 mm, vias 1 -> 0
- net /ESP_TX: track 35.4 -> 35.7 mm, vias 1 -> 0
- net GND: track 3.84 -> 3.95 mm, vias 0 -> 8

Commit message: Update Routing
Parts:
- moved R1 25.8 mm to (227.2, 105.2)
- moved R10 11.7 mm to (191.7, 92.5)
Routing:
- net +5V: track 20.0 -> 34.2 mm, vias 1 -> 2
- net /OUTPUT_ENABLE: track 25.8 -> 40.0 mm
- net /SW_1: track 66.9 -> 53.4 mm
- net +3V3: track 90.5 -> 97.1 mm, vias 8 -> 23
- net /ESP_EN: track 42.7 -> 37.2 mm
- net GND: track 3.95 -> 9.27 mm, vias 8 -> 15
- net /BOOT: track 27.1 -> 26.5 mm
- added copper zone on B.Cu, net +3V3
