File: Hardware Files/8Bit_WiFi_Visualizer.sch (KiCad schematic (older format))
At the start: 34 parts, among them J1 USB_B_Micro, J2 Conn_01x04, SW1 SW_Push_Dual, SW2 SW_SPST, SW3 SW_SPST, U1 3.3V 1A, U2 74HC595, U3 ESP-WROOM-02D

Commit message: Cleanup Schematic
Connections:
- wire segments 126 -> 125
Other:
- note added: "Programming Header"
- moved on the sheet: C2, C3, C4, C5, C6, D1, D2, D3, D4, D5, D6, D7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

Commit message: Change to 1206 components and reroute
Parts:
- removed R2, R3, R4, R5, R6, R7, R8, R9: 75R, Resistor_SMD:R_0805_2012Metric, symbol Device:R
- added J1, J2: Conn_01x01, MountingHole:MountingHole_3.2mm_M3_DIN965_Pad, symbol Connector_Generic:Conn_01x01
- C2, C3, C4, C5, C6: footprint Capacitor_SMD:C_0805_2012Metric -> Capacitor_SMD:C_1206_3216Metric_Pad1.42x1.75mm_HandSolder
- D1, D2, D3, D4, D5, D6, D7, D8: footprint LED_SMD:LED_0805_2012Metric_Castellated -> LED_SMD:LED_1206_3216Metric_Pad1.42x1.75mm_HandSolder
- R1, R10, R11, R12, R13: footprint Resistor_SMD:R_0805_2012Metric -> Resistor_SMD:R_1206_3216Metric_Pad1.42x1.75mm_HandSolder
Connections:
- wire segments 125 -> 121
Other:
- moved on the sheet: R13

Commit message: change components to 1206 footprints and remove some components
Parts:
- renumbered J1 to J3, J2 to J4
Changed lines of the file:
@@
 Text Label 8700 1650 0    50   ~ 0
 CLOCK
-Text Label 4050 3825 2    50   ~ 0
+Text Label 3600 3875 2    50   ~ 0
 CLOCK
 Text Label 3550 4475 2    50   ~ 0
@@
 	2950 4375 3950 4375
 $Comp
-L Connector_Generic:Conn_01x01 J1
+L Connector_Generic:Conn_01x01 J3
 U 1 1 5F7C5A4F
 P 12450 1600
-F 0 "J1" H 12530 1642 50  0000 L CNN
+F 0 "J3" H 12530 1642 50  0000 L CNN
 F 1 "Conn_01x01" H 12530 1551 50  0000 L CNN
 F 2 "MountingHole:MountingHole_3.2mm_M3_DIN965_Pad" H 12450 1600 50  0001 C CNN
@@
 $EndComp
 $Comp
-L Connector_Generic:Conn_01x01 J2
+L Connector_Generic:Conn_01x01 J4
 U 1 1 5F7C66A3
 P 12450 1800
-F 0 "J2" H 12530 1842 50  0000 L CNN
+F 0 "J4" H 12530 1842 50  0000 L CNN
 F 1 "Conn_01x01" H 12530 1751 50  0000 L CNN
 F 2 "MountingHole:MountingHole_3.2mm_M3_DIN965_Pad" H 12450 1800 50  0001 C CNN
@@
 $EndComp
 $Comp
-L power:GND #PWR?
+L power:GND #PWR0107
 U 1 1 5F7C69AE
 P 12075 1925
-F 0 "#PWR?" H 12075 1675 50  0001 C CNN
+F 0 "#PWR0107" H 12075 1675 50  0001 C CNN
 F 1 "GND" H 12080 1752 50  0000 C CNN
 F 2 "" H 12075 1925 50  0001 C CNN

Commit message: Re-Annotate Schematic
Parts:
- renumbered C3 to C1, C4 to C3, C5 to C4, C6 to C5, R12 to R1, R11 to R2, R10 to R3, R13 to R4, R1 to R5
Changed lines of the file:
@@
 Wire Wire Line
 	3425 7000 3425 7150
-$Comp
-L Device:R R1
-U 1 1 5DD4F5D4
-P 2475 6450
-F 0 "R1" H 2545 6496 50  0000 L CNN
-F 1 "10k" H 2545 6405 50  0000 L CNN
-F 2 "Resistor_SMD:R_1206_3216Metric_Pad1.42x1.75mm_HandSolder" V 2405 6450 50  0001 C CNN
-F 3 "~" H 2475 6450 50  0001 C CNN
-F 4 "RC0805JR-0710KL" H 2475 6450 50  0001 C CNN "Manufacturer PN"
-	1    2475 6450
-	1    0    0    -1
-$EndComp
 Text Label 1825 6800 0    50   ~ 0
 SW_1
@@
 	1500 3775 2000 3775
 $Comp
-L Device:C_Small C4
+L Device:C_Small C3
 U 1 1 5DD4DF71
 P 1050 4575
-F 0 "C4" H 1142 4621 50  0000 L CNN
+F 0 "C3" H 1142 4621 50  0000 L CNN
 F 1 "10uF" H 1142 4530 50  0000 L CNN
 F 2 "Capacitor_SMD:C_1206_3216Metric_Pad1.42x1.75mm_HandSolder" H 1050 4575 50  0001 C CNN
@@
 $EndComp
 $Comp
-L Device:C_Small C5
+L Device:C_Small C4
 U 1 1 5DD55927
 P 1450 4575
-F 0 "C5" H 1542 4621 50  0000 L CNN
+F 0 "C4" H 1542 4621 50  0000 L CNN
 F 1 "0.1uF" H 1542 4530 50  0000 L CNN
 F 2 "Capacitor_SMD:C_1206_3216Metric_Pad1.42x1.75mm_HandSolder" H 1450 4575 50  0001 C CNN
@@
 	1050 4725 1450 4725
 $Comp
-L Device:C_Small C6
+L Device:C_Small C5
 U 1 1 5DD84BF8
 P 6525 1875
-F 0 "C6" H 6617 1921 50  0000 L CNN
+F 0 "C5" H 6617 1921 50  0000 L CNN
 F 1 "0.1uF" H 6617 1830 50  0000 L CNN
 F 2 "Capacitor_SMD:C_1206_3216Metric_Pad1.42x1.75mm_HandSolder" H 6525 1875 50  0001 C CNN
@@
 	1    6525 1875
 	1    0    0    -1
-$EndComp
-$Comp
-L Device:R R11
-U 1 1 5DD8941C
-P 6525 1375
-F 0 "R11" H 6595 1421 50  0000 L CNN
-F 1 "10k" H 6595 1330 50  0000 L CNN
-F 2 "Resistor_SMD:R_1206_3216Metric_Pad1.42x1.75mm_HandSolder" V 6455 1375 50  0001 C CNN
-F 3 "~" H 6525 1375 50  0001 C CNN
-F 4 "RC0805JR-0710KL" H 6525 1375 50  0001 C CNN "Manufacturer PN"
-	1    6525 1375
-	-1   0    0    -1
 $EndComp
 $Comp
@@
 ESP_EN
 $Comp
-L Device:R R13
+L Device:R R4
 U 1 1 5DDC28A2
 P 3950 4525
-F 0 "R13" H 4020 4571 50  0000 L CNN
+F 0 "R4" H 4020 4571 50  0000 L CNN
 F 1 "10k" H 4020 4480 50  0000 L CNN
 F 2 "Resistor_SMD:R_1206_3216Metric_Pad1.42x1.75mm_HandSolder" V 3880 4525 50  0001 C CNN
@@
 $EndComp
 $Comp
-L Device:C_Small C3
+L Device:C_Small C1
 U 1 1 5DE4618C
 P 2200 1500
-F 0 "C3" H 2292 1546 50  0000 L CNN
+F 0 "C1" H 2292 1546 50  0000 L CNN
 F 1 "4.7uF" H 2292 1455 50  0000 L CNN
 F 2 "Capacitor_SMD:C_1206_3216Metric_Pad1.42x1.75mm_HandSolder" H 2200 1500 50  0001 C CNN
@@
 BOOT
 $Comp
-L Device:R R12
+L Device:R R1
 U 1 1 5DDDB6FD
 P 5275 1375
-F 0 "R12" H 5345 1421 50  0000 L CNN
+F 0 "R1" H 5345 1421 50  0000 L CNN
 F 1 "10k" H 5345 1330 50  0000 L CNN
 F 2 "Resistor_SMD:R_1206_3216Metric_Pad1.42x1.75mm_HandSolder" V 5205 1375 50  0001 C CNN
@@
 $EndComp
 $Comp
-L Device:R R10
+L Device:R R3
 U 1 1 5DD4919D
 P 8675 2300
-F 0 "R10" H 8745 2346 50  0000 L CNN
+F 0 "R3" H 8745 2346 50  0000 L CNN
 F 1 "10k" H 8745 2255 50  0000 L CNN
 F 2 "Resistor_SMD:R_1206_3216Metric_Pad1.42x1.75mm_HandSolder" V 8605 2300 50  0001 C CNN
@@
 	12075 1600 12250 1600
 Connection ~ 12075 1800
+$Comp
+L Device:R R2
+U 1 1 5DD8941C
+P 6525 1375
+F 0 "R2" H 6595 1421 50  0000 L CNN
+F 1 "10k" H 6595 1330 50  0000 L CNN
+F 2 "Resistor_SMD:R_1206_3216Metric_Pad1.42x1.75mm_HandSolder" V 6455 1375 50  0001 C CNN
+F 3 "~" H 6525 1375 50  0001 C CNN
+F 4 "RC0805JR-0710KL" H 6525 1375 50  0001 C CNN "Manufacturer PN"
+	1    6525 1375
+	-1   0    0    -1
+$EndComp
+$Comp
+L Device:R R5
+U 1 1 5DD4F5D4
+P 2475 6450
+F 0 "R5" H 2545 6496 50  0000 L CNN
+F 1 "10k" H 2545 6405 50  0000 L CNN
+F 2 "Resistor_SMD:R_1206_3216Metric_Pad1.42x1.75mm_HandSolder" V 2405 6450 50  0001 C CNN
+F 3 "~" H 2475 6450 50  0001 C CNN
+F 4 "RC0805JR-0710KL" H 2475 6450 50  0001 C CNN "Manufacturer PN"
+	1    2475 6450
+	1    0    0    -1
+$EndComp
 $EndSCHEMATC

Commit message: Scrub BOM details
Parts:
- C1, C2: Manufacturer PN CC0805ZRY5V6BB475 -> (none)
- C3: Manufacturer PN CC0805ZKY5V5BB106 -> (none)
- C4, C5: Manufacturer PN CC0805ZRY5V9BB104 -> (none)
- D1, D2, D3, D4, D5, D6, D7, D8: Manufacturer PN LH R974-LP-1 -> (none)
- J1: Manufacturer PN 1050170001 -> (none)
- R1, R2, R3, R4, R5: Manufacturer PN RC0805JR-0710KL -> (none)
- SW1: Manufacturer PN PTS645SK50SMTR92 LFS -> (none)
- SW2, SW3: Manufacturer PN PTS636 SM25F SMTR LFS -> (none)
- U1: Manufacturer PN AP2114H-3.3TRG1 -> (none)
- U2: Manufacturer PN SN74HC595DR -> (none)
Changed lines of the file:
@@
 F 2 "LED_SMD:LED_1206_3216Metric_Pad1.42x1.75mm_HandSolder" H 9725 3875 50  0001 C CNN
 F 3 "~" H 9725 3875 50  0001 C CNN
-F 4 "LH R974-LP-1" H 9725 3875 50  0001 C CNN "Manufacturer PN"
+F 4 "" H 9725 3875 50  0001 C CNN "Manufacturer PN"
 	1    9725 3875
 	0    -1   -1   0
@@
 F 2 "LED_SMD:LED_1206_3216Metric_Pad1.42x1.75mm_HandSolder" H 9325 3875 50  0001 C CNN
 F 3 "~" H 9325 3875 50  0001 C CNN
-F 4 "LH R974-LP-1" H 9325 3875 50  0001 C CNN "Manufacturer PN"
+F 4 "" H 9325 3875 50  0001 C CNN "Manufacturer PN"
 	1    9325 3875
 	0    -1   -1   0
@@
 F 2 "LED_SMD:LED_1206_3216Metric_Pad1.42x1.75mm_HandSolder" H 8925 3875 50  0001 C CNN
 F 3 "~" H 8925 3875 50  0001 C CNN
-F 4 "LH R974-LP-1" H 8925 3875 50  0001 C CNN "Manufacturer PN"
+F 4 "" H 8925 3875 50  0001 C CNN "Manufacturer PN"
 	1    8925 3875
 	0    -1   -1   0
@@
 F 2 "LED_SMD:LED_1206_3216Metric_Pad1.42x1.75mm_HandSolder" H 8525 3875 50  0001 C CNN
 F 3 "~" H 8525 3875 50  0001 C CNN
-F 4 "LH R974-LP-1" H 8525 3875 50  0001 C CNN "Manufacturer PN"
+F 4 "" H 8525 3875 50  0001 C CNN "Manufacturer PN"
 	1    8525 3875
 	0    -1   -1   0
@@
 F 2 "LED_SMD:LED_1206_3216Metric_Pad1.42x1.75mm_HandSolder" H 8125 3875 50  0001 C CNN
 F 3 "~" H 8125 3875 50  0001 C CNN
-F 4 "LH R974-LP-1" H 8125 3875 50  0001 C CNN "Manufacturer PN"
+F 4 "" H 8125 3875 50  0001 C CNN "Manufacturer PN"
 	1    8125 3875
 	0    -1   -1   0
@@
 F 2 "LED_SMD:LED_1206_3216Metric_Pad1.42x1.75mm_HandSolder" H 7725 3875 50  0001 C CNN
 F 3 "~" H 7725 3875 50  0001 C CNN
-F 4 "LH R974-LP-1" H 7725 3875 50  0001 C CNN "Manufacturer PN"
+F 4 "" H 7725 3875 50  0001 C CNN "Manufacturer PN"
 	1    7725 3875
 	0    -1   -1   0
@@
 F 2 "LED_SMD:LED_1206_3216Metric_Pad1.42x1.75mm_HandSolder" H 7325 3875 50  0001 C CNN
 F 3 "~" H 7325 3875 50  0001 C CNN
-F 4 "LH R974-LP-1" H 7325 3875 50  0001 C CNN "Manufacturer PN"
+F 4 "" H 7325 3875 50  0001 C CNN "Manufacturer PN"
 	1    7325 3875
 	0    -1   -1   0
@@
 F 2 "LED_SMD:LED_1206_3216Metric_Pad1.42x1.75mm_HandSolder" H 10125 3875 50  0001 C CNN
 F 3 "~" H 10125 3875 50  0001 C CNN
-F 4 "LH R974-LP-1" H 10125 3875 50  0001 C CNN "Manufacturer PN"
+F 4 "" H 10125 3875 50  0001 C CNN "Manufacturer PN"
 	1    10125 3875
 	0    -1   -1   0
@@
 F 2 "8Bit_WiFi_Visualizer_Footprints:PTS645SK50SMTR92LFS" H 2975 7000 50  0001 C CNN
 F 3 "~" H 2975 7000 50  0001 C CNN
-F 4 "PTS645SK50SMTR92 LFS" H 2975 6800 50  0001 C CNN "Manufacturer PN"
+F 4 "" H 2975 6800 50  0001 C CNN "Manufacturer PN"
 	1    2975 6800
 	1    0    0    -1
@@
 F 2 "Capacitor_SMD:C_1206_3216Metric_Pad1.42x1.75mm_HandSolder" H 1050 4575 50  0001 C CNN
 F 3 "~" H 1050 4575 50  0001 C CNN
-F 4 "CC0805ZKY5V5BB106" H 1050 4575 50  0001 C CNN "Manufacturer PN"
+F 4 "" H 1050 4575 50  0001 C CNN "Manufacturer PN"
 	1    1050 4575
 	1    0    0    -1
@@
 F 2 "Capacitor_SMD:C_1206_3216Metric_Pad1.42x1.75mm_HandSolder" H 1450 4575 50  0001 C CNN
 F 3 "~" H 1450 4575 50  0001 C CNN
-F 4 "CC0805ZRY5V9BB104" H 1450 4575 50  0001 C CNN "Manufacturer PN"
+F 4 "" H 1450 4575 50  0001 C CNN "Manufacturer PN"
 	1    1450 4575
 	1    0    0    -1
@@
 F 2 "Capacitor_SMD:C_1206_3216Metric_Pad1.42x1.75mm_HandSolder" H 6525 1875 50  0001 C CNN
 F 3 "~" H 6525 1875 50  0001 C CNN
-F 4 "CC0805ZRY5V9BB104" H 6525 1875 50  0001 C CNN "Manufacturer PN"
+F 4 "" H 6525 1875 50  0001 C CNN "Manufacturer PN"
 	1    6525 1875
 	1    0    0    -1
@@
 F 2 "Resistor_SMD:R_1206_3216Metric_Pad1.42x1.75mm_HandSolder" V 3880 4525 50  0001 C CNN
 F 3 "~" H 3950 4525 50  0001 C CNN
-F 4 "RC0805JR-0710KL" H 3950 4525 50  0001 C CNN "Manufacturer PN"
+F 4 "" H 3950 4525 50  0001 C CNN "Manufacturer PN"
 	1    3950 4525
 	-1   0    0    -1
@@
 F 2 "8Bit_WiFi_Visualizer_Footprints:USB_Micro-B_Molex-105017-0001_3D" H 1625 1450 50  0001 C CNN
 F 3 "~" H 1625 1450 50  0001 C CNN
-F 4 "1050170001" H 1475 1500 50  0001 C CNN "Manufacturer PN"
+F 4 "" H 1475 1500 50  0001 C CNN "Manufacturer PN"
 	1    1475 1500
 	1    0    0    -1
@@
 F 2 "Package_TO_SOT_SMD:SOT-223-3_TabPin2" H 2900 1500 50  0001 C CNN
 F 3 "https://www.diodes.com/assets/Datasheets/AP2114.pdf" H 3000 1050 50  0001 C CNN
-F 4 "AP2114H-3.3TRG1" H 2900 1300 50  0001 C CNN "Manufacturer PN"
+F 4 "" H 2900 1300 50  0001 C CNN "Manufacturer PN"
 	1    2900 1300
 	1    0    0    -1
@@
 F 2 "Capacitor_SMD:C_1206_3216Metric_Pad1.42x1.75mm_HandSolder" H 2200 1500 50  0001 C CNN
 F 3 "~" H 2200 1500 50  0001 C CNN
-F 4 "CC0805ZRY5V6BB475" H 2200 1500 50  0001 C CNN "Manufacturer PN"
+F 4 "" H 2200 1500 50  0001 C CNN "Manufacturer PN"
 	1    2200 1500
 	1    0    0    -1
@@
 F 2 "Capacitor_SMD:C_1206_3216Metric_Pad1.42x1.75mm_HandSolder" H 3550 1500 50  0001 C CNN
 F 3 "~" H 3550 1500 50  0001 C CNN
-F 4 "CC0805ZRY5V6BB475" H 3550 1500 50  0001 C CNN "Manufacturer PN"
+F 4 "" H 3550 1500 50  0001 C CNN "Manufacturer PN"
 	1    3550 1500
 	1    0    0    -1
@@
 F 2 "8Bit_WiFi_Visualizer_Footprints:PTS636_SM25F_SMTR_LFS" H 7150 1650 50  0001 C CNN
 F 3 "file:///C:/Users/A552123/Documents/KiCad%20Projects/beginner_project_1/beginner_project_1_footprint_library.pretty/datasheet.pdf" H 7150 1650 50  0001 C CNN
-F 4 "PTS636 SM25F SMTR LFS" H 7150 1650 50  0001 C CNN "Manufacturer PN"
+F 4 "" H 7150 1650 50  0001 C CNN "Manufacturer PN"
 	1    7150 1650
 	1    0    0    -1
@@
 F 2 "8Bit_WiFi_Visualizer_Footprints:PTS636_SM25F_SMTR_LFS" H 5625 1700 50  0001 C CNN
 F 3 "file:///C:/Users/A552123/Documents/KiCad%20Projects/beginner_project_1/beginner_project_1_footprint_library.pretty/datasheet.pdf" H 5625 1700 50  0001 C CNN
-F 4 "PTS636 SM25F SMTR LFS" H 5625 1700 50  0001 C CNN "Manufacturer PN"
+F 4 "" H 5625 1700 50  0001 C CNN "Manufacturer PN"
 	1    5625 1700
 	1    0    0    -1
@@
 F 2 "Resistor_SMD:R_1206_3216Metric_Pad1.42x1.75mm_HandSolder" V 5205 1375 50  0001 C CNN
 F 3 "~" H 5275 1375 50  0001 C CNN
-F 4 "RC0805JR-0710KL" H 5275 1375 50  0001 C CNN "Manufacturer PN"
+F 4 "" H 5275 1375 50  0001 C CNN "Manufacturer PN"
 	1    5275 1375
 	-1   0    0    -1
@@
 F 2 "Package_SO:SOIC-16_3.9x9.9mm_P1.27mm" H 9725 1850 50  0001 C CNN
 F 3 "http://www.ti.com/lit/ds/symlink/sn74hc595.pdf" H 9725 1850 50  0001 C CNN
-F 4 "SN74HC595DR" H 9725 1850 50  0001 C CNN "Manufacturer PN"
+F 4 "" H 9725 1850 50  0001 C CNN "Manufacturer PN"
 	1    9725 1850
 	1    0    0    -1
@@
 F 2 "Resistor_SMD:R_1206_3216Metric_Pad1.42x1.75mm_HandSolder" V 8605 2300 50  0001 C CNN
 F 3 "~" H 8675 2300 50  0001 C CNN
-F 4 "RC0805JR-0710KL" H 8675 2300 50  0001 C CNN "Manufacturer PN"
+F 4 "" H 8675 2300 50  0001 C CNN "Manufacturer PN"
 	1    8675 2300
 	-1   0    0    1
@@
 F 2 "Resistor_SMD:R_1206_3216Metric_Pad1.42x1.75mm_HandSolder" V 6455 1375 50  0001 C CNN
 F 3 "~" H 6525 1375 50  0001 C CNN
-F 4 "RC0805JR-0710KL" H 6525 1375 50  0001 C CNN "Manufacturer PN"
+F 4 "" H 6525 1375 50  0001 C CNN "Manufacturer PN"
 	1    6525 1375
 	-1   0    0    -1
@@
 F 2 "Resistor_SMD:R_1206_3216Metric_Pad1.42x1.75mm_HandSolder" V 2405 6450 50  0001 C CNN
 F 3 "~" H 2475 6450 50  0001 C CNN
-F 4 "RC0805JR-0710KL" H 2475 6450 50  0001 C CNN "Manufacturer PN"
+F 4 "" H 2475 6450 50  0001 C CNN "Manufacturer PN"
 	1    2475 6450
 	1    0    0    -1

Commit message: Add descriptions
Parts:
- C1, C2: Description (none) -> 4.7 uF 1206 Capacitor
- C3: Description (none) -> 10uF 1206 Capacitor
- C4, C5: Description (none) -> 0.1uF 1206 Capacitor
- D1, D2, D3, D4, D5, D6, D7, D8: Description (none) -> 3.2V 1206 LED
- J1: Description (none) -> MicroUSB Connector SMD
- J2: Description (none) -> 2.54mm Male PCB Header
- J3, J4: Description (none) -> Mounting Holes
- R1, R2, R3, R4, R5: Description (none) -> 10k 1206 Resistor
- U1: Description (none) -> 3.3V 1A SOT223 LDO Linear Regulator
- U2: Description (none) -> Shift Register SOIC 16
- U3: Description (none) -> ESP 8266 SMD Module
Changed lines of the file:
@@
 F 3 "~" H 9725 3875 50  0001 C CNN
 F 4 "" H 9725 3875 50  0001 C CNN "Manufacturer PN"
+F 5 "3.2V 1206 LED" H 9725 3875 50  0001 C CNN "Description"
 	1    9725 3875
 	0    -1   -1   0
@@
 F 3 "~" H 9325 3875 50  0001 C CNN
 F 4 "" H 9325 3875 50  0001 C CNN "Manufacturer PN"
+F 5 "3.2V 1206 LED" H 9325 3875 50  0001 C CNN "Description"
 	1    9325 3875
 	0    -1   -1   0
@@
 F 3 "~" H 8925 3875 50  0001 C CNN
 F 4 "" H 8925 3875 50  0001 C CNN "Manufacturer PN"
+F 5 "3.2V 1206 LED" H 8925 3875 50  0001 C CNN "Description"
 	1    8925 3875
 	0    -1   -1   0
@@
 F 3 "~" H 8525 3875 50  0001 C CNN
 F 4 "" H 8525 3875 50  0001 C CNN "Manufacturer PN"
+F 5 "3.2V 1206 LED" H 8525 3875 50  0001 C CNN "Description"
 	1    8525 3875
 	0    -1   -1   0
@@
 F 3 "~" H 8125 3875 50  0001 C CNN
 F 4 "" H 8125 3875 50  0001 C CNN "Manufacturer PN"
+F 5 "3.2V 1206 LED" H 8125 3875 50  0001 C CNN "Description"
 	1    8125 3875
 	0    -1   -1   0
@@
 F 3 "~" H 7725 3875 50  0001 C CNN
 F 4 "" H 7725 3875 50  0001 C CNN "Manufacturer PN"
+F 5 "3.2V 1206 LED" H 7725 3875 50  0001 C CNN "Description"
 	1    7725 3875
 	0    -1   -1   0
@@
 F 3 "~" H 7325 3875 50  0001 C CNN
 F 4 "" H 7325 3875 50  0001 C CNN "Manufacturer PN"
+F 5 "3.2V 1206 LED" H 7325 3875 50  0001 C CNN "Description"
 	1    7325 3875
 	0    -1   -1   0
@@
 F 3 "~" H 10125 3875 50  0001 C CNN
 F 4 "" H 10125 3875 50  0001 C CNN "Manufacturer PN"
+F 5 "3.2V 1206 LED" H 10125 3875 50  0001 C CNN "Description"
 	1    10125 3875
 	0    -1   -1   0
@@
 F 3 "~" H 1050 4575 50  0001 C CNN
 F 4 "" H 1050 4575 50  0001 C CNN "Manufacturer PN"
+F 5 "10uF 1206 Capacitor" H 1050 4575 50  0001 C CNN "Description"
 	1    1050 4575
 	1    0    0    -1
@@
 F 3 "~" H 1450 4575 50  0001 C CNN
 F 4 "" H 1450 4575 50  0001 C CNN "Manufacturer PN"
+F 5 "0.1uF 1206 Capacitor" H 1450 4575 50  0001 C CNN "Description"
 	1    1450 4575
 	1    0    0    -1
@@
 F 3 "~" H 6525 1875 50  0001 C CNN
 F 4 "" H 6525 1875 50  0001 C CNN "Manufacturer PN"
+F 5 "0.1uF 1206 Capacitor" H 6525 1875 50  0001 C CNN "Description"
 	1    6525 1875
 	1    0    0    -1
@@
 F 3 "~" H 3950 4525 50  0001 C CNN
 F 4 "" H 3950 4525 50  0001 C CNN "Manufacturer PN"
+F 5 "10k 1206 Resistor" H 3950 4525 50  0001 C CNN "Description"
 	1    3950 4525
 	-1   0    0    -1
@@
 F 3 "~" H 1625 1450 50  0001 C CNN
 F 4 "" H 1475 1500 50  0001 C CNN "Manufacturer PN"
+F 5 "MicroUSB Connector SMD" H 1475 1500 50  0001 C CNN "Description"
 	1    1475 1500
 	1    0    0    -1
@@
 F 3 "https://www.diodes.com/assets/Datasheets/AP2114.pdf" H 3000 1050 50  0001 C CNN
 F 4 "" H 2900 1300 50  0001 C CNN "Manufacturer PN"
+F 5 "3.3V 1A SOT223 LDO Linear Regulator" H 2900 1300 50  0001 C CNN "Description"
 	1    2900 1300
 	1    0    0    -1
@@
 F 3 "~" H 2200 1500 50  0001 C CNN
 F 4 "" H 2200 1500 50  0001 C CNN "Manufacturer PN"
+F 5 "4.7 uF 1206 Capacitor" H 2200 1500 50  0001 C CNN "Description"
 	1    2200 1500
 	1    0    0    -1
@@
 F 3 "~" H 3550 1500 50  0001 C CNN
 F 4 "" H 3550 1500 50  0001 C CNN "Manufacturer PN"
+F 5 "4.7 uF 1206 Capacitor" H 3550 1500 50  0001 C CNN "Description"
 	1    3550 1500
 	1    0    0    -1
@@
 F 3 "~" H 5275 1375 50  0001 C CNN
 F 4 "" H 5275 1375 50  0001 C CNN "Manufacturer PN"
+F 5 "10k 1206 Resistor" H 5275 1375 50  0001 C CNN "Description"
 	1    5275 1375
 	-1   0    0    -1
@@
 F 3 "http://www.ti.com/lit/ds/symlink/sn74hc595.pdf" H 9725 1850 50  0001 C CNN
 F 4 "" H 9725 1850 50  0001 C CNN "Manufacturer PN"
+F 5 "Shift Register SOIC 16" H 9725 1850 50  0001 C CNN "Description"
 	1    9725 1850
 	1    0    0    -1
@@
 F 2 "Connector_PinHeader_2.54mm:PinHeader_1x04_P2.54mm_Vertical" H 5225 6300 50  0001 C CNN
 F 3 "~" H 5225 6300 50  0001 C CNN
+F 4 "2.54mm Male PCB Header" H 5225 6300 50  0001 C CNN "Description"
 	1    5225 6300
 	-1   0    0    -1
@@
 F 3 "~" H 8675 2300 50  0001 C CNN
 F 4 "" H 8675 2300 50  0001 C CNN "Manufacturer PN"
+F 5 "10k 1206 Resistor" H 8675 2300 50  0001 C CNN "Description"
 	1    8675 2300
 	-1   0    0    1
@@
 F 3 "https://www.espressif.com/sites/default/files/documentation/esp-wroom-02u_esp-wroom-02d_datasheet_en.pdf" H 2150 6125 50  0001 C CNN
 F 4 "ESP-WROOM-02D" H 2100 4825 50  0001 C CNN "Manufacturer PN"
+F 5 "ESP 8266 SMD Module" H 2100 4825 50  0001 C CNN "Description"
 	1    2100 4825
 	1    0    0    -1
@@
 F 2 "MountingHole:MountingHole_3.2mm_M3_DIN965_Pad" H 12450 1600 50  0001 C CNN
 F 3 "~" H 12450 1600 50  0001 C CNN
+F 4 "Mounting Holes" H 12450 1600 50  0001 C CNN "Description"
 	1    12450 1600
 	1    0    0    -1
@@
 F 2 "MountingHole:MountingHole_3.2mm_M3_DIN965_Pad" H 12450 1800 50  0001 C CNN
 F 3 "~" H 12450 1800 50  0001 C CNN
+F 4 "Mounting Holes" H 12450 1800 50  0001 C CNN "Description"
 	1    12450 1800
 	1    0    0    -1
@@
 F 3 "~" H 6525 1375 50  0001 C CNN
 F 4 "" H 6525 1375 50  0001 C CNN "Manufacturer PN"
+F 5 "10k 1206 Resistor" H 6525 1375 50  0001 C CNN "Description"
 	1    6525 1375
 	-1   0    0    -1
@@
 F 3 "~" H 2475 6450 50  0001 C CNN
 F 4 "" H 2475 6450 50  0001 C CNN "Manufacturer PN"
+F 5 "10k 1206 Resistor" H 2475 6450 50  0001 C CNN "Description"
 	1    2475 6450
 	1    0    0    -1

Commit message: update part numbers
Parts:
- C1, C2: LCSC Order Number (none) -> C1872; Manufacturer (none) -> Samsung Electro-Mechanics; Manufacturer PN (none) -> CL31B475KAHNNNE
- C3: LCSC Order Number (none) -> C318763; Manufacturer (none) -> Samsung Electro-Mechanics; Manufacturer PN (none) -> CL31A106MAHNNNE
- C4, C5: LCSC Order Number (none) -> C24497; Manufacturer (none) -> Samsung Electro-Mechanics; Manufacturer PN (none) -> CL31B104KBCNNNC
- D1, D2, D3, D4, D5, D6, D7, D8: LCSC Order Number (none) -> C125088; Manufacturer (none) -> Lite-On; Manufacturer PN (none) -> LTST-C150TBKT
- J1: LCSC Order Number (none) -> 1050170001; Manufacturer (none) -> MOLEX; Manufacturer PN (none) -> C136000
- R1, R2, R3, R4, R5: LCSC Order Number (none) -> C136460; Manufacturer (none) -> YAGEO; Manufacturer PN (none) -> RC1206JR-0710KL
- SW1: Description (none) -> SPST 50mA @ 12VDC Vertical Round Button SMD,6x6x5mm Tactile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; LCSC Order Number (none) -> C255812; Manufacturer (none) -> Hongyuan Precision; Manufacturer PN (none) -> 1TS005F-2500-5001
- SW2, SW3: Description (none) -> SPST 50mA @ 12VDC SMD,6x3.5x5mm; LCSC Order Number (none) -> C318844; Manufacturer (none) -> Hongyuan Precision; Manufacturer PN (none) -> 1TS002B-2700-5000-CT
- U1: LCSC Order Number (none) -> C92102; Manufacturer (none) -> Diodes Incorporated; Manufacturer PN (none) -> AZ1117CH-3.3TRG1
- U2: LCSC Order Number (none) -> C5947; Manufacturer (none) -> Nexperia; Manufacturer PN (none) -> 74HC595D,118
- U3: LCSC Order Number (none) -> C473007; Manufacturer (none) -> Espressif Systems
