File: Hardware Files/8Bit_WiFi_Visualizer.sch (KiCad schematic (older format))
At the start: 28 parts, among them J1 USB_B_Micro, J2 Conn_01x04, J3 Conn_01x01, J4 Conn_01x01, SW1 SW_Push_Dual, SW2 SW_SPST, SW3 SW_SPST, U1 3.3V 1A, U2 74HC595, U3 ESP-WROOM-02D

Commit message: fix USB MPN
Parts:
- D1, D2, D3, D4, D5, D6, D7, D8: Manufacturer Lite-On -> Lite-On
- J1: LCSC Order Number 1050170001 -> C136000; Manufacturer MOLEX -> MOLEX; Manufacturer PN C136000 -> 1050170001
Changed lines of the file:
@@
 F 5 "3.2V 1206 LED" H 9725 3875 50  0001 C CNN "Description"
 F 6 "	C125088" H 9725 3875 50  0001 C CNN "LCSC Order Number"
-F 7 "	Lite-On" H 9725 3875 50  0001 C CNN "Manufacturer"
+F 7 "Lite-On" H 9725 3875 50  0001 C CNN "Manufacturer"
 	1    9725 3875
 	0    -1   -1   0
@@
 F 5 "3.2V 1206 LED" H 9325 3875 50  0001 C CNN "Description"
 F 6 "	C125088" H 9325 3875 50  0001 C CNN "LCSC Order Number"
-F 7 "	Lite-On" H 9325 3875 50  0001 C CNN "Manufacturer"
+F 7 "Lite-On" H 9325 3875 50  0001 C CNN "Manufacturer"
 	1    9325 3875
 	0    -1   -1   0
@@
 F 5 "3.2V 1206 LED" H 8925 3875 50  0001 C CNN "Description"
 F 6 "	C125088" H 8925 3875 50  0001 C CNN "LCSC Order Number"
-F 7 "	Lite-On" H 8925 3875 50  0001 C CNN "Manufacturer"
+F 7 "Lite-On" H 8925 3875 50  0001 C CNN "Manufacturer"
 	1    8925 3875
 	0    -1   -1   0
@@
 F 5 "3.2V 1206 LED" H 8525 3875 50  0001 C CNN "Description"
 F 6 "	C125088" H 8525 3875 50  0001 C CNN "LCSC Order Number"
-F 7 "	Lite-On" H 8525 3875 50  0001 C CNN "Manufacturer"
+F 7 "Lite-On" H 8525 3875 50  0001 C CNN "Manufacturer"
 	1    8525 3875
 	0    -1   -1   0
@@
 F 5 "3.2V 1206 LED" H 8125 3875 50  0001 C CNN "Description"
 F 6 "	C125088" H 8125 3875 50  0001 C CNN "LCSC Order Number"
-F 7 "	Lite-On" H 8125 3875 50  0001 C CNN "Manufacturer"
+F 7 "Lite-On" H 8125 3875 50  0001 C CNN "Manufacturer"
 	1    8125 3875
 	0    -1   -1   0
@@
 F 5 "3.2V 1206 LED" H 7725 3875 50  0001 C CNN "Description"
 F 6 "	C125088" H 7725 3875 50  0001 C CNN "LCSC Order Number"
-F 7 "	Lite-On" H 7725 3875 50  0001 C CNN "Manufacturer"
+F 7 "Lite-On" H 7725 3875 50  0001 C CNN "Manufacturer"
 	1    7725 3875
 	0    -1   -1   0
@@
 F 5 "3.2V 1206 LED" H 7325 3875 50  0001 C CNN "Description"
 F 6 "	C125088" H 7325 3875 50  0001 C CNN "LCSC Order Number"
-F 7 "	Lite-On" H 7325 3875 50  0001 C CNN "Manufacturer"
+F 7 "Lite-On" H 7325 3875 50  0001 C CNN "Manufacturer"
 	1    7325 3875
 	0    -1   -1   0
@@
 F 5 "3.2V 1206 LED" H 10125 3875 50  0001 C CNN "Description"
 F 6 "	C125088" H 10125 3875 50  0001 C CNN "LCSC Order Number"
-F 7 "	Lite-On" H 10125 3875 50  0001 C CNN "Manufacturer"
+F 7 "Lite-On" H 10125 3875 50  0001 C CNN "Manufacturer"
 	1    10125 3875
 	0    -1   -1   0
@@
 F 2 "8Bit_WiFi_Visualizer_Footprints:USB_Micro-B_Molex-105017-0001_3D" H 1625 1450 50  0001 C CNN
 F 3 "~" H 1625 1450 50  0001 C CNN
-F 4 "	C136000" H 1475 1500 50  0001 C CNN "Manufacturer PN"
+F 4 "1050170001" H 1475 1500 50  0001 C CNN "Manufacturer PN"
 F 5 "MicroUSB Connector SMD" H 1475 1500 50  0001 C CNN "Description"
-F 6 "	1050170001" H 1475 1500 50  0001 C CNN "LCSC Order Number"
-F 7 "	MOLEX" H 1475 1500 50  0001 C CNN "Manufacturer"
+F 6 "C136000" H 1475 1500 50  0001 C CNN "LCSC Order Number"
+F 7 "MOLEX" H 1475 1500 50  0001 C CNN "Manufacturer"
 	1    1475 1500
 	1    0    0    -1
