File: Hardware Files/8Bit_WiFi_Visualizer.sch (KiCad schematic (older format))
At the start: 28 parts, among them J1 USB_B_Micro, J2 Conn_01x04, J3 Conn_01x01, J4 Conn_01x01, SW1 SW_Push_Dual, SW2 SW_SPST, SW3 SW_SPST, U1 3.3V 1A, U2 74HC595, U3 ESP-WROOM-02D

Commit message: Change capacitors to 1uF
Parts:
- C1, C2: value 4.7uF -> 1uF; Description 4.7 uF 1206 Capacitor -> 1 uF 1206 Capacitor; LCSC Order Number C1872 -> C13832; Manufacturer PN CL31B475KAHNNNE -> CL31B105KCHNNNE
- C3: LCSC Order Number C318763 -> C14860; Manufacturer PN CL31A106MAHNNNE -> CL31B106KAHNNNE
- C4, C5: value 0.1uF -> 1uF; Description 0.1uF 1206 Capacitor -> 1 uF 1206 Capacitor; LCSC Order Number C24497 -> C13832; Manufacturer PN CL31B104KBCNNNC -> CL31B105KCHNNNE
- D1, D2, D3, D4, D5, D6, D7, D8: LCSC Order Number C125088 -> C125088
Changed lines of the file:
@@
 F 4 "LTST-C150TBKT" H 9725 3875 50  0001 C CNN "Manufacturer PN"
 F 5 "3.2V 1206 LED" H 9725 3875 50  0001 C CNN "Description"
-F 6 "	C125088" H 9725 3875 50  0001 C CNN "LCSC Order Number"
+F 6 "C125088" H 9725 3875 50  0001 C CNN "LCSC Order Number"
 F 7 "Lite-On" H 9725 3875 50  0001 C CNN "Manufacturer"
 	1    9725 3875
@@
 F 4 "LTST-C150TBKT" H 9325 3875 50  0001 C CNN "Manufacturer PN"
 F 5 "3.2V 1206 LED" H 9325 3875 50  0001 C CNN "Description"
-F 6 "	C125088" H 9325 3875 50  0001 C CNN "LCSC Order Number"
+F 6 "C125088" H 9325 3875 50  0001 C CNN "LCSC Order Number"
 F 7 "Lite-On" H 9325 3875 50  0001 C CNN "Manufacturer"
 	1    9325 3875
@@
 F 4 "LTST-C150TBKT" H 8925 3875 50  0001 C CNN "Manufacturer PN"
 F 5 "3.2V 1206 LED" H 8925 3875 50  0001 C CNN "Description"
-F 6 "	C125088" H 8925 3875 50  0001 C CNN "LCSC Order Number"
+F 6 "C125088" H 8925 3875 50  0001 C CNN "LCSC Order Number"
 F 7 "Lite-On" H 8925 3875 50  0001 C CNN "Manufacturer"
 	1    8925 3875
@@
 F 4 "LTST-C150TBKT" H 8525 3875 50  0001 C CNN "Manufacturer PN"
 F 5 "3.2V 1206 LED" H 8525 3875 50  0001 C CNN "Description"
-F 6 "	C125088" H 8525 3875 50  0001 C CNN "LCSC Order Number"
+F 6 "C125088" H 8525 3875 50  0001 C CNN "LCSC Order Number"
 F 7 "Lite-On" H 8525 3875 50  0001 C CNN "Manufacturer"
 	1    8525 3875
@@
 F 4 "LTST-C150TBKT" H 8125 3875 50  0001 C CNN "Manufacturer PN"
 F 5 "3.2V 1206 LED" H 8125 3875 50  0001 C CNN "Description"
-F 6 "	C125088" H 8125 3875 50  0001 C CNN "LCSC Order Number"
+F 6 "C125088" H 8125 3875 50  0001 C CNN "LCSC Order Number"
 F 7 "Lite-On" H 8125 3875 50  0001 C CNN "Manufacturer"
 	1    8125 3875
@@
 F 4 "LTST-C150TBKT" H 7725 3875 50  0001 C CNN "Manufacturer PN"
 F 5 "3.2V 1206 LED" H 7725 3875 50  0001 C CNN "Description"
-F 6 "	C125088" H 7725 3875 50  0001 C CNN "LCSC Order Number"
+F 6 "C125088" H 7725 3875 50  0001 C CNN "LCSC Order Number"
 F 7 "Lite-On" H 7725 3875 50  0001 C CNN "Manufacturer"
 	1    7725 3875
@@
 F 4 "LTST-C150TBKT" H 7325 3875 50  0001 C CNN "Manufacturer PN"
 F 5 "3.2V 1206 LED" H 7325 3875 50  0001 C CNN "Description"
-F 6 "	C125088" H 7325 3875 50  0001 C CNN "LCSC Order Number"
+F 6 "C125088" H 7325 3875 50  0001 C CNN "LCSC Order Number"
 F 7 "Lite-On" H 7325 3875 50  0001 C CNN "Manufacturer"
 	1    7325 3875
@@
 F 4 "LTST-C150TBKT" H 10125 3875 50  0001 C CNN "Manufacturer PN"
 F 5 "3.2V 1206 LED" H 10125 3875 50  0001 C CNN "Description"
-F 6 "	C125088" H 10125 3875 50  0001 C CNN "LCSC Order Number"
+F 6 "C125088" H 10125 3875 50  0001 C CNN "LCSC Order Number"
 F 7 "Lite-On" H 10125 3875 50  0001 C CNN "Manufacturer"
 	1    10125 3875
@@
 F 2 "Capacitor_SMD:C_1206_3216Metric_Pad1.42x1.75mm_HandSolder" H 1050 4575 50  0001 C CNN
 F 3 "~" H 1050 4575 50  0001 C CNN
-F 4 "CL31A106MAHNNNE" H 1050 4575 50  0001 C CNN "Manufacturer PN"
+F 4 "CL31B106KAHNNNE" H 1050 4575 50  0001 C CNN "Manufacturer PN"
 F 5 "10uF 1206 Capacitor" H 1050 4575 50  0001 C CNN "Description"
-F 6 "C318763" H 1050 4575 50  0001 C CNN "LCSC Order Number"
+F 6 "C14860" H 1050 4575 50  0001 C CNN "LCSC Order Number"
 F 7 "Samsung Electro-Mechanics" H 1050 4575 50  0001 C CNN "Manufacturer"
 	1    1050 4575
@@
 P 1450 4575
 F 0 "C4" H 1542 4621 50  0000 L CNN
-F 1 "0.1uF" H 1542 4530 50  0000 L CNN
+F 1 "1uF" H 1542 4530 50  0000 L CNN
 F 2 "Capacitor_SMD:C_1206_3216Metric_Pad1.42x1.75mm_HandSolder" H 1450 4575 50  0001 C CNN
 F 3 "~" H 1450 4575 50  0001 C CNN
-F 4 "CL31B104KBCNNNC" H 1450 4575 50  0001 C CNN "Manufacturer PN"
-F 5 "0.1uF 1206 Capacitor" H 1450 4575 50  0001 C CNN "Description"
-F 6 "C24497" H 1450 4575 50  0001 C CNN "LCSC Order Number"
+F 4 "CL31B105KCHNNNE" H 1450 4575 50  0001 C CNN "Manufacturer PN"
+F 5 "1 uF 1206 Capacitor" H 1450 4575 50  0001 C CNN "Description"
+F 6 "C13832" H 1450 4575 50  0001 C CNN "LCSC Order Number"
 F 7 "Samsung Electro-Mechanics" H 1450 4575 50  0001 C CNN "Manufacturer"
 	1    1450 4575
@@
 P 6525 1875
 F 0 "C5" H 6617 1921 50  0000 L CNN
-F 1 "0.1uF" H 6617 1830 50  0000 L CNN
+F 1 "1uF" H 6617 1830 50  0000 L CNN
 F 2 "Capacitor_SMD:C_1206_3216Metric_Pad1.42x1.75mm_HandSolder" H 6525 1875 50  0001 C CNN
 F 3 "~" H 6525 1875 50  0001 C CNN
-F 4 "CL31B104KBCNNNC" H 6525 1875 50  0001 C CNN "Manufacturer PN"
-F 5 "0.1uF 1206 Capacitor" H 6525 1875 50  0001 C CNN "Description"
-F 6 "C24497" H 6525 1875 50  0001 C CNN "LCSC Order Number"
+F 4 "CL31B105KCHNNNE" H 6525 1875 50  0001 C CNN "Manufacturer PN"
+F 5 "1 uF 1206 Capacitor" H 6525 1875 50  0001 C CNN "Description"
+F 6 "C13832" H 6525 1875 50  0001 C CNN "LCSC Order Number"
 F 7 "Samsung Electro-Mechanics" H 6525 1875 50  0001 C CNN "Manufacturer"
 	1    6525 1875
@@
 P 2200 1500
 F 0 "C1" H 2292 1546 50  0000 L CNN
-F 1 "4.7uF" H 2292 1455 50  0000 L CNN
+F 1 "1uF" H 2292 1455 50  0000 L CNN
 F 2 "Capacitor_SMD:C_1206_3216Metric_Pad1.42x1.75mm_HandSolder" H 2200 1500 50  0001 C CNN
 F 3 "~" H 2200 1500 50  0001 C CNN
-F 4 "CL31B475KAHNNNE" H 2200 1500 50  0001 C CNN "Manufacturer PN"
-F 5 "4.7 uF 1206 Capacitor" H 2200 1500 50  0001 C CNN "Description"
-F 6 "C1872" H 2200 1500 50  0001 C CNN "LCSC Order Number"
+F 4 "CL31B105KCHNNNE" H 2200 1500 50  0001 C CNN "Manufacturer PN"
+F 5 "1 uF 1206 Capacitor" H 2200 1500 50  0001 C CNN "Description"
+F 6 "C13832" H 2200 1500 50  0001 C CNN "LCSC Order Number"
 F 7 "Samsung Electro-Mechanics" H 2200 1500 50  0001 C CNN "Manufacturer"
 	1    2200 1500
@@
 P 3550 1500
 F 0 "C2" H 3642 1546 50  0000 L CNN
-F 1 "4.7uF" H 3642 1455 50  0000 L CNN
+F 1 "1uF" H 3642 1455 50  0000 L CNN
 F 2 "Capacitor_SMD:C_1206_3216Metric_Pad1.42x1.75mm_HandSolder" H 3550 1500 50  0001 C CNN
 F 3 "~" H 3550 1500 50  0001 C CNN
-F 4 "CL31B475KAHNNNE" H 3550 1500 50  0001 C CNN "Manufacturer PN"
-F 5 "4.7 uF 1206 Capacitor" H 3550 1500 50  0001 C CNN "Description"
-F 6 "C1872" H 3550 1500 50  0001 C CNN "LCSC Order Number"
+F 4 "CL31B105KCHNNNE" H 3550 1500 50  0001 C CNN "Manufacturer PN"
+F 5 "1 uF 1206 Capacitor" H 3550 1500 50  0001 C CNN "Description"
+F 6 "C13832" H 3550 1500 50  0001 C CNN "LCSC Order Number"
 F 7 "Samsung Electro-Mechanics" H 3550 1500 50  0001 C CNN "Manufacturer"
 	1    3550 1500

Commit message: Change USB connector and update revision
Parts:
- J1: footprint 8Bit_WiFi_Visualizer_Footprints:USB_Micro-B_Molex-105017-0001_3D -> 8Bit_WiFi_Visualizer_Footprints:U-F-M5DD-Y-L; LCSC Order Number C136000 -> C91146; Manufacturer MOLEX -> Korean Hroparts Elec; Manufacturer PN 1050170001 -> U-F-M5DD-Y-L
Changed lines of the file:
@@
 F 0 "J1" H 1532 1967 50  0000 C CNN
 F 1 "USB_B_Micro" H 1532 1876 50  0000 C CNN
-F 2 "8Bit_WiFi_Visualizer_Footprints:USB_Micro-B_Molex-105017-0001_3D" H 1625 1450 50  0001 C CNN
+F 2 "8Bit_WiFi_Visualizer_Footprints:U-F-M5DD-Y-L" H 1625 1450 50  0001 C CNN
 F 3 "~" H 1625 1450 50  0001 C CNN
-F 4 "1050170001" H 1475 1500 50  0001 C CNN "Manufacturer PN"
+F 4 "U-F-M5DD-Y-L" H 1475 1500 50  0001 C CNN "Manufacturer PN"
 F 5 "MicroUSB Connector SMD" H 1475 1500 50  0001 C CNN "Description"
-F 6 "C136000" H 1475 1500 50  0001 C CNN "LCSC Order Number"
-F 7 "MOLEX" H 1475 1500 50  0001 C CNN "Manufacturer"
+F 6 "C91146" H 1475 1500 50  0001 C CNN "LCSC Order Number"
+F 7 "Korean Hroparts Elec" H 1475 1500 50  0001 C CNN "Manufacturer"
 	1    1475 1500
 	1    0    0    -1

Commit message: rearrange Schematic
Connections:
- wire segments 121 -> 120
Other:
- note removed: "External pull down on GPIO15\nfor boot options"
- note removed: "Programming Header"
- moved on the sheet: C3, C4, D1, D2, D3, D4, D5, D6, D7, D8, J2, R3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
